Commit message: changes to upper and lower limits

File: src/arcs3r21v2_description/urdf/arcs3r21v2.xacro (robot description, xacro)
@@ -149,5 +149,5 @@
   <child link="link1_1"/>
   <axis xyz="-0.0 -0.0 1.0"/>
-  <limit upper="6.283185" lower="0.0" effort="100" velocity="100"/>
+  <limit upper="6.33552" lower="-6.33552" effort="100" velocity="100"/>
 </joint>
 <joint name="rev2" type="revolute">
@@ -156,5 +156,5 @@
   <child link="link2_1"/>
   <axis xyz="0.0 -1.0 0.0"/>
-  <limit upper="6.283185" lower="0.0" effort="100" velocity="100"/>
+  <limit upper="6.33552" lower="-6.33552" effort="100" velocity="100"/>
 </joint>
 <joint name="rev3" type="revolute">
@@ -163,5 +163,5 @@
   <child link="link3_1"/>
   <axis xyz="0.0 -1.0 0.0"/>
-  <limit upper="6.283185" lower="0.0" effort="100" velocity="100"/>
+  <limit upper="6.33552" lower="-6.33552" effort="100" velocity="100"/>
 </joint>
 <joint name="rev4" type="revolute">
@@ -170,5 +170,5 @@
   <child link="link4_1"/>
   <axis xyz="-0.0 1.0 -0.0"/>
-  <limit upper="6.283185" lower="0.0" effort="100" velocity="100"/>
+  <limit upper="6.33552" lower="-6.33552" effort="100" velocity="100"/>
 </joint>
 <joint name="rev5" type="revolute">
@@ -177,5 +177,5 @@
   <child link="link5_1"/>
   <axis xyz="-0.0 -0.0 1.0"/>
-  <limit upper="6.283185" lower="0.0" effort="100" velocity="100"/>
+  <limit upper="6.33552" lower="-6.33552" effort="100" velocity="100"/>
 </joint>
 <joint name="rev6" type="revolute">
@@ -184,5 +184,5 @@
   <child link="link6_1"/>
   <axis xyz="0.0 -1.0 0.0"/>
-  <limit upper="6.283185" lower="0.0" effort="100" velocity="100"/>
+  <limit upper="6.33552" lower="-6.33552" effort="100" velocity="100"/>
 </joint>
 </robot>
