Commit message: robot simple move1

File: install/arcs3r21v2_description/share/arcs3r21v2_description/urdf/arcs3r21v2.xacro (robot description, xacro)
@@ -1,188 +1 @@
-<?xml version="1.0" ?>
-<robot name="arcs3r21v2" xmlns:xacro="http://www.ros.org/wiki/xacro">
-<xacro:include filename="$(find arcs3r21v2_description)/urdf/materials.xacro" />
-<xacro:include filename="$(find arcs3r21v2_description)/urdf/arcs3r21v2.trans" />
-<xacro:include filename="$(find arcs3r21v2_description)/urdf/arcs3r21v2.gazebo" />
-<link name="base_link">
-  <inertial>
-    <origin xyz="-0.019489127148037858 -0.004507096530095732 0.06890832828660853" rpy="0 0 0"/>
-    <mass value="0.3581512769045181"/>
-    <inertia ixx="0.000533" iyy="0.00055" izz="0.000655" ixy="-0.0" iyz="9e-06" ixz="0.0"/>
-  </inertial>
-  <visual>
-    <origin xyz="0 0 0" rpy="0 0 0"/>
-    <geometry>
-      <mesh filename="file://$(find arcs3r21v2_description)/meshes/base_link.stl" scale="0.001 0.001 0.001"/>
-    </geometry>
-    <material name="silver"/>
-  </visual>
-  <collision>
-    <origin xyz="0 0 0" rpy="0 0 0"/>
-    <geometry>
-      <mesh filename="file://$(find arcs3r21v2_description)/meshes/base_link.stl" scale="0.001 0.001 0.001"/>
-    </geometry>
-  </collision>
-</link>
-<link name="link1_1">
-  <inertial>
-    <origin xyz="2.7189135486348215e-06 0.006511138704688911 0.06951856212512914" rpy="0 0 0"/>
-    <mass value="1.1817680983524481"/>
-    <inertia ixx="0.002691" iyy="0.002499" izz="0.001645" ixy="0.0" iyz="-1.5e-05" ixz="-0.0"/>
-  </inertial>
-  <visual>
-    <origin xyz="0.019508 0.005227 -0.100081" rpy="0 0 0"/>
-    <geometry>
-      <mesh filename="file://$(find arcs3r21v2_description)/meshes/link1_1.stl" scale="0.001 0.001 0.001"/>
-    </geometry>
-    <material name="silver"/>
-  </visual>
-  <collision>
-    <origin xyz="0.019508 0.005227 -0.100081" rpy="0 0 0"/>
-    <geometry>
-      <mesh filename="file://$(find arcs3r21v2_description)/meshes/link1_1.stl" scale="0.001 0.001 0.001"/>
-    </geometry>
-  </collision>
-</link>
-<link name="link2_1">
-  <inertial>
-    <origin xyz="-0.12092661465022866 0.06680849598485737 -5.725962811120588e-07" rpy="0 0 0"/>
-    <mass value="2.987553170242043"/>
-    <inertia ixx="0.004898" iyy="0.038087" izz="0.03974" ixy="-0.000898" iyz="0.0" ixz="1e-06"/>
-  </inertial>
-  <visual>
-    <origin xyz="0.019508 -0.055573 -0.167281" rpy="0 0 0"/>
-    <geometry>
-      <mesh filename="file://$(find arcs3r21v2_description)/meshes/link2_1.stl" scale="0.001 0.001 0.001"/>
-    </geometry>
-    <material name="silver"/>
-  </visual>
-  <collision>
-    <origin xyz="0.019508 -0.055573 -0.167281" rpy="0 0 0"/>
-    <geometry>
-      <mesh filename="file://$(find arcs3r21v2_description)/meshes/link2_1.stl" scale="0.001 0.001 0.001"/>
-    </geometry>
-  </collision>
-</link>
-<link name="link3_1">
-  <inertial>
-    <origin xyz="-0.1347210042850771 -0.049548544656501436 -4.016904008419253e-06" rpy="0 0 0"/>
-    <mass value="1.8351757406943898"/>
-    <inertia ixx="0.001964" iyy="0.018868" izz="0.01933" ixy="-0.001206" iyz="-0.0" ixz="1e-06"/>
-  </inertial>
-  <visual>
-    <origin xyz="0.289508 -0.055473 -0.167281" rpy="0 0 0"/>
-    <geometry>
-      <mesh filename="file://$(find arcs3r21v2_description)/meshes/link3_1.stl" scale="0.001 0.001 0.001"/>
-    </geometry>
-    <material name="silver"/>
-  </visual>
-  <collision>
-    <origin xyz="0.289508 -0.055473 -0.167281" rpy="0 0 0"/>
-    <geometry>
-      <mesh filename="file://$(find arcs3r21v2_description)/meshes/link3_1.stl" scale="0.001 0.001 0.001"/>
-    </geometry>
-  </collision>
-</link>
-<link name="link4_1">
-  <inertial>
-    <origin xyz="1.8338933284178793e-06 0.06644523303963622 -0.0046808621407556095" rpy="0 0 0"/>
-    <mass value="0.7526945620031449"/>
-    <inertia ixx="0.001427" iyy="0.00091" izz="0.00108" ixy="-0.0" iyz="5.8e-05" ixz="0.0"/>
-  </inertial>
-  <visual>
-    <origin xyz="0.547008 -0.053773 -0.167281" rpy="0 0 0"/>
-    <geometry>
-      <mesh filename="file://$(find arcs3r21v2_description)/meshes/link4_1.stl" scale="0.001 0.001 0.001"/>
-    </geometry>
-    <material name="silver"/>
-  </visual>
-  <collision>
-    <origin xyz="0.547008 -0.053773 -0.167281" rpy="0 0 0"/>
-    <geometry>
-      <mesh filename="file://$(find arcs3r21v2_description)/meshes/link4_1.stl" scale="0.001 0.001 0.001"/>
-    </geometry>
-  </collision>
-</link>
-<link name="link5_1">
-  <inertial>
-    <origin xyz="2.3665292054886322e-06 0.00607101118430009 0.04253930344379153" rpy="0 0 0"/>
-    <mass value="0.5803090573673972"/>
-    <inertia ixx="0.000836" iyy="0.000493" izz="0.00078" ixy="-0.0" iyz="-8e-06" ixz="-0.0"/>
-  </inertial>
-  <visual>
-    <origin xyz="0.547008 -0.139273 -0.216281" rpy="0 0 0"/>
-    <geometry>
-      <mesh filename="file://$(find arcs3r21v2_description)/meshes/link5_1.stl" scale="0.001 0.001 0.001"/>
-    </geometry>
-    <material name="silver"/>
-  </visual>
-  <collision>
-    <origin xyz="0.547008 -0.139273 -0.216281" rpy="0 0 0"/>
-    <geometry>
-      <mesh filename="file://$(find arcs3r21v2_description)/meshes/link5_1.stl" scale="0.001 0.001 0.001"/>
-    </geometry>
-  </collision>
-</link>
-<link name="link6_1">
-  <inertial>
-    <origin xyz="-2.0425992675043858e-08 -0.019893414223481648 -0.0001503824488282013" rpy="0 0 0"/>
-    <mass value="0.17860634529456432"/>
-    <inertia ixx="8.7e-05" iyy="0.000127" izz="8.8e-05" ixy="-0.0" iyz="-0.0" ixz="0.0"/>
-  </inertial>
-  <visual>
-    <origin xyz="0.547008 -0.090273 -0.263781" rpy="0 0 0"/>
-    <geometry>
-      <mesh filename="file://$(find arcs3r21v2_description)/meshes/link6_1.stl" scale="0.001 0.001 0.001"/>
-    </geometry>
-    <material name="silver"/>
-  </visual>
-  <collision>
-    <origin xyz="0.547008 -0.090273 -0.263781" rpy="0 0 0"/>
-    <geometry>
-      <mesh filename="file://$(find arcs3r21v2_description)/meshes/link6_1.stl" scale="0.001 0.001 0.001"/>
-    </geometry>
-  </collision>
-</link>
-<joint name="rev1" type="revolute">
-  <origin xyz="-0.019508 -0.005227 0.100081" rpy="0 0 0"/>
-  <parent link="base_link"/>
-  <child link="link1_1"/>
-  <axis xyz="-0.0 -0.0 1.0"/>
-  <limit upper="6.283185" lower="0.0" effort="100" velocity="100"/>
-</joint>
-<joint name="rev2" type="revolute">
-  <origin xyz="0.0 0.0608 0.0672" rpy="0 0 0"/>
-  <parent link="link1_1"/>
-  <child link="link2_1"/>
-  <axis xyz="0.0 -1.0 0.0"/>
-  <limit upper="6.283185" lower="0.0" effort="100" velocity="100"/>
-</joint>
-<joint name="rev3" type="revolute">
-  <origin xyz="-0.27 -0.0001 0.0" rpy="0 0 0"/>
-  <parent link="link2_1"/>
-  <child link="link3_1"/>
-  <axis xyz="0.0 -1.0 0.0"/>
-  <limit upper="6.283185" lower="0.0" effort="100" velocity="100"/>
-</joint>
-<joint name="rev4" type="revolute">
-  <origin xyz="-0.2575 -0.0017 0.0" rpy="0 0 0"/>
-  <parent link="link3_1"/>
-  <child link="link4_1"/>
-  <axis xyz="-0.0 1.0 -0.0"/>
-  <limit upper="6.283185" lower="0.0" effort="100" velocity="100"/>
-</joint>
-<joint name="rev5" type="revolute">
-  <origin xyz="0.0 0.0855 0.049" rpy="0 0 0"/>
-  <parent link="link4_1"/>
-  <child link="link5_1"/>
-  <axis xyz="-0.0 -0.0 1.0"/>
-  <limit upper="6.283185" lower="0.0" effort="100" velocity="100"/>
-</joint>
-<joint name="rev6" type="revolute">
-  <origin xyz="0.0 -0.049 0.0475" rpy="0 0 0"/>
-  <parent link="link5_1"/>
-  <child link="link6_1"/>
-  <axis xyz="0.0 -1.0 0.0"/>
-  <limit upper="6.283185" lower="0.0" effort="100" velocity="100"/>
-</joint>
-</robot>
+/home/amos/cs_ws/build/arcs3r21v2_description/urdf/arcs3r21v2.xacro

File: install/arcs3r21v2_description/share/arcs3r21v2_description/urdf/materials.xacro (robot description, xacro)
@@ -1,6 +1 @@
-<?xml version="1.0" ?>
-<robot name="arcs3r21v2" xmlns:xacro="http://www.ros.org/wiki/xacro" >
-<material name="silver">
-  <color rgba="0.700 0.700 0.700 1.000"/>
-</material>
-</robot>
+/home/amos/cs_ws/build/arcs3r21v2_description/urdf/materials.xacro
